Commit message: Updated pipette_tool and pipette_tip description.

File: urdf/pipette_tool.xacro (robot description, xacro)
@@ -5,12 +5,12 @@
   connected_to
   ">
-    <xacro:property name="pipette_offset" value="0.110" />
-    <xacro:property name="tcp_offset" value="0.083" />
+    <xacro:property name="pipette_tool_offset" value="0.111" />
+    <xacro:property name="pipette_tip_offset" value="0.119" />
+    <xacro:property name="tcp_offset" value="0.001" />
     <link name="${ur_type}_pipette_tool">
       <visual>
         <geometry>
-          <mesh filename="package://titration_robot_cell_description/meshes/one1000.stl" scale="0.001 0.001 0.001" />
+          <mesh filename="package://titration_robot_cell_description/meshes/one200.stl" scale="0.001 0.001 0.001" />
         </geometry>
-        <!-- <origin rpy="0 0 0" xyz="0 0 0"/> -->
         <origin rpy="${-pi/2} 0 ${-pi/2}" xyz="0 0 0"/>
         <material name="grey"/>
@@ -18,8 +18,22 @@
       <collision>
         <geometry>
-          <mesh filename="package://titration_robot_cell_description/meshes/one1000.stl" scale="0.001 0.001 0.001" />
+          <mesh filename="package://titration_robot_cell_description/meshes/one200.stl" scale="0.001 0.001 0.001" />
         </geometry>
-        <!-- <origin rpy="0 0 0" xyz="0 0 0"/> -->
         <origin rpy="${-pi/2} 0 ${-pi/2}" xyz="0 0 0"/>
+      </collision>
+    </link>
+    <link name="${ur_type}_pipette_tip">
+      <visual>
+        <geometry>
+          <mesh filename="package://titration_robot_cell_description/meshes/pipette_tip.stl" scale="0.001 0.001 0.001" />
+        </geometry>
+        <origin rpy="${-pi/2} 0 0" xyz="0 0 0"/>
+        <material name="white"/>
+      </visual>
+      <collision>
+        <geometry>
+          <mesh filename="package://titration_robot_cell_description/meshes/pipette_tip.stl" scale="0.001 0.001 0.001" />
+        </geometry>
+        <origin rpy="${-pi/2} 0 0" xyz="0 0 0"/>
       </collision>
     </link>
@@ -28,9 +42,13 @@
       <parent link="${ur_type}_${connected_to}"/>
       <child link="${ur_type}_pipette_tool"/>
-      <!-- <origin rpy="${-pi/2} 0 ${-pi/2}" xyz="0 0 ${pipette_offset}"/> -->
-      <origin xyz="0 0 ${pipette_offset}" rpy="0 0 0"/>
+      <origin xyz="0 0 ${pipette_tool_offset}" rpy="0 0 0"/>
+    </joint>
+    <joint name="${ur_type}_pipette_tip_joint" type="fixed">
+      <parent link="${ur_type}_pipette_tool"/>
+      <child link="${ur_type}_pipette_tip"/>
+      <origin xyz="0 0 ${pipette_tip_offset}" rpy="0 0 0"/>
     </joint>
     <joint name="${ur_type}_tcp_joint" type="fixed">
-      <parent link="${ur_type}_pipette_tool"/>
+      <parent link="${ur_type}_pipette_tip"/>
       <child link="${ur_type}_tcp"/>
       <origin xyz="0 0 ${tcp_offset}" rpy="0 0 0"/>

Commit message: Updated to beaker_600ml, pipette_tool distance to ur5_tool, stirrer model.

File: urdf/pipette_tool.xacro (robot description, xacro)
@@ -5,5 +5,5 @@
   connected_to
   ">
-    <xacro:property name="pipette_tool_offset" value="0.111" />
+    <xacro:property name="pipette_tool_offset" value="0.116" />
     <xacro:property name="pipette_tip_offset" value="0.119" />
     <xacro:property name="tcp_offset" value="0.001" />

File: urdf/titration_robot_cell_macro.xacro (robot description, xacro)
@@ -34,6 +34,8 @@
     <xacro:property name="wall_offset" value="0.75" />
     <xacro:property name="table_beaker_offset" value="0.01" />
-    <xacro:property name="table_stirrer_offset" value="0.01" />
-    <xacro:property name="stirrer_height" value="0.057" />
+    <xacro:property name="stirrer_width" value="0.210" />
+    <xacro:property name="stirrer_depth" value="0.320" />
+    <xacro:property name="stirrer_height" value="0.105" />
+    <xacro:property name="table_stirrer_offset" value="0.0525" />
     <xacro:property name="meter_width" value="0.096" />
     <xacro:property name="meter_depth" value="0.112" />
@@ -75,5 +77,5 @@
       <visual>
         <geometry>
-          <mesh filename="package://titration_robot_cell_description/meshes/beaker.stl" scale="0.01 0.01 0.01" />
+          <mesh filename="package://titration_robot_cell_description/meshes/beaker_600ml.stl" scale="0.001 0.001 0.001" />
         </geometry>
         <origin rpy="0 0 0" xyz="0 0 0"/>
@@ -82,5 +84,5 @@
       <collision>
         <geometry>
-          <mesh filename="package://titration_robot_cell_description/meshes/beaker.stl" scale="0.01 0.01 0.01"/>
+          <mesh filename="package://titration_robot_cell_description/meshes/beaker_600ml.stl" scale="0.001 0.001 0.001"/>
         </geometry>
         <origin rpy="0 0 0" xyz="0 0 0"/>
@@ -90,5 +92,5 @@
       <visual>
         <geometry>
-          <mesh filename="package://titration_robot_cell_description/meshes/stirrer.stl" scale="0.001 0.001 0.001" />
+          <box size="${stirrer_depth} ${stirrer_width} ${stirrer_height}"/>
         </geometry>
         <origin rpy="0 0 0" xyz="0 0 0"/>
@@ -97,5 +99,5 @@
       <collision>
         <geometry>
-          <mesh filename="package://titration_robot_cell_description/meshes/stirrer.stl" scale="0.001 0.001 0.001"/>
+          <box size="${stirrer_width} ${stirrer_depth} ${stirrer_height}"/>
         </geometry>
         <origin rpy="0 0 0" xyz="0 0 0"/>
@@ -105,5 +107,5 @@
       <visual>
         <geometry>
-          <mesh filename="package://titration_robot_cell_description/meshes/beaker.stl" scale="0.01 0.01 0.01" />
+          <mesh filename="package://titration_robot_cell_description/meshes/beaker_600ml.stl" scale="0.001 0.001 0.001" />
         </geometry>
         <origin rpy="0 0 0" xyz="0 0 0"/>
@@ -112,5 +114,5 @@
       <collision>
         <geometry>
-          <mesh filename="package://titration_robot_cell_description/meshes/beaker.stl" scale="0.01 0.01 0.01"/>
+          <mesh filename="package://titration_robot_cell_description/meshes/beaker_600ml.stl" scale="0.001 0.001 0.001"/>
         </geometry>
         <origin rpy="0 0 0" xyz="0 0 0"/>
@@ -167,15 +169,15 @@
       <parent link="table"/>
       <child link="stirrer"/>
-      <origin xyz="${table_width/4+0.185} ${table_width/4} ${table_height/2+table_stirrer_offset}" rpy="${pi/2} 0 ${pi/2}" />
+      <origin xyz="${table_width/4} ${table_width/4} ${table_height/2+table_stirrer_offset}" rpy="0 0 0" />
     </joint>
     <joint name="table_to_beaker_analyte" type="fixed">
       <parent link="table"/>
       <child link="beaker_analyte"/>
-      <origin xyz="${table_width/4} ${table_width/4} ${table_height/2+table_beaker_offset+stirrer_height}" rpy="${pi/2} 0 0" />
+      <origin xyz="${table_width/4} ${table_width/4} ${table_height/2+table_beaker_offset+stirrer_height+0.001}" rpy="${pi/2} 0 0" />
     </joint>
     <joint name="table_to_ph_meter" type="fixed">
       <parent link="table"/>
       <child link="ph_meter"/>
-      <origin xyz="0 ${table_width/4} ${table_height/2+meter_width/2}" rpy="0 0 0" />
+      <origin xyz="${-table_width/4} ${table_width/4} ${table_height/2+meter_width/2}" rpy="0 0 0" />
     </joint>
     <joint name="beaker_analyte_to_ph_probe" type="fixed">
