Commit message: Added retort_stand. Updated stirrer model. Edited ph_meter position.

File: urdf/titration_robot_cell_macro.xacro (robot description, xacro)
@@ -25,4 +25,7 @@
     <material name="light_purple">
       <color rgba="0.80 0.76 0.89 0.75"/>
+    </material>
+    <material name="light_red">
+      <color rgba="1 0 0 0.5"/>
     </material>
     <xacro:property name="table_width" value="0.9" />
@@ -44,4 +47,5 @@
     <xacro:property name="probe_height_offset" value="0.100" />
     <xacro:property name="probe_radial_offset" value="0.025" />
+    <xacro:property name="retort_y_offset" value="0.078" />
     <link name="wall">
       <visual>
@@ -99,5 +103,5 @@
       <collision>
         <geometry>
-          <box size="${stirrer_width} ${stirrer_depth} ${stirrer_height}"/>
+          <box size="${stirrer_depth} ${stirrer_width} ${stirrer_height}"/>
         </geometry>
         <origin rpy="0 0 0" xyz="0 0 0"/>
@@ -140,11 +144,26 @@
         </geometry>
         <origin rpy="0 0 0" xyz="0 0 0"/>
+        <material name="light_red"/>
+      </visual>
+      <collision>
+        <geometry>
+          <cylinder radius="${probe_diameter/2}" length="${probe_length}"/>
+        </geometry>
+        <origin rpy="0 0 0" xyz="0 0 0"/>
+      </collision>
+    </link>
+    <link name="retort_stand">
+      <visual>
+        <geometry>
+          <mesh filename="package://titration_robot_cell_description/meshes/retort_stand.stl" scale="0.001 0.001 0.001" />
+        </geometry>
+        <origin rpy="${pi/2} 0 0" xyz="0 0 0"/>
         <material name="grey"/>
       </visual>
       <collision>
         <geometry>
-          <cylinder radius="${probe_diameter/2}" length="${probe_length}"/>
-        </geometry>
-        <origin rpy="0 0 0" xyz="0 0 0"/>
+          <mesh filename="package://titration_robot_cell_description/meshes/retort_stand.stl" scale="0.001 0.001 0.001"/>
+        </geometry>
+        <origin rpy="${pi/2} 0 0" xyz="0 0 0"/>
       </collision>
     </link>
@@ -179,5 +198,5 @@
       <parent link="table"/>
       <child link="ph_meter"/>
-      <origin xyz="${-table_width/4} ${table_width/4} ${table_height/2+meter_width/2}" rpy="0 0 0" />
+      <origin xyz="${-table_width/8} 0 ${table_height/2+meter_width/2}" rpy="0 0 0" />
     </joint>
     <joint name="beaker_analyte_to_ph_probe" type="fixed">
@@ -185,4 +204,9 @@
       <child link="ph_probe"/>
       <origin xyz="0 ${probe_height_offset} ${-probe_radial_offset}" rpy="${-pi/2} 0 0" />
+    </joint>
+    <joint name="table_to_retort_stand" type="fixed">
+      <parent link="table"/>
+      <child link="retort_stand"/>
+      <origin xyz="0 ${table_width/4+retort_y_offset} ${table_height/2}" rpy="0 0 0" />
     </joint>
     <joint name="table_to_robot_mount" type="fixed">

Commit message: Added invisible left and right barrier.

File: urdf/titration_robot_cell_macro.xacro (robot description, xacro)
@@ -16,4 +16,7 @@
     <material name="grey">
       <color rgba="0.5 0.5 0.5 1"/>
+    </material>
+    <material name="invisible">
+      <color rgba="0.9 0.9 0.9 0.1"/>
     </material>
     <material name="white">
@@ -78,4 +81,34 @@
       </collision>
     </link>
+    <link name="right_barrier">
+      <visual>
+        <geometry>
+          <box size="${table_width} 0.005 ${table_height}"/>
+        </geometry>
+        <origin rpy="0 0 0" xyz="0 0 0"/>
+        <material name="invisible"/>
+      </visual>
+      <collision>
+        <geometry>
+          <box size="${table_width} 0.005 ${table_height}"/>
+        </geometry>
+        <origin rpy="0 0 0" xyz="0 0 0"/>
+      </collision>
+    </link>
+    <link name="left_barrier">
+      <visual>
+        <geometry>
+          <box size="${table_width} 0.005 ${table_height}"/>
+        </geometry>
+        <origin rpy="0 0 0" xyz="0 0 0"/>
+        <material name="invisible"/>
+      </visual>
+      <collision>
+        <geometry>
+          <box size="${table_width} 0.005 ${table_height}"/>
+        </geometry>
+        <origin rpy="0 0 0" xyz="0 0 0"/>
+      </collision>
+    </link>
     <link name="beaker_titrant">
       <visual>
@@ -180,5 +213,15 @@
       <origin xyz="0 0 ${table_height/2}" rpy="0 0 0" />
     </joint>
-    <joint name="table_to_beaker_titrant" type="fixed">
+    <joint name="table_to_right_barrier" type="fixed">
+      <parent link="table"/>
+      <child link="right_barrier"/>
+      <origin xyz="0 ${-table_width/2+0.050} ${table_height}" rpy="0 0 0" />
+    </joint>
+    <joint name="table_to_left_barrier" type="fixed">
+      <parent link="table"/>
+      <child link="left_barrier"/>
+      <origin xyz="0 ${table_width/2-0.050} ${table_height}" rpy="0 0 0" />
+    </joint>
+     <joint name="table_to_beaker_titrant" type="fixed">
       <parent link="table"/>
       <child link="beaker_titrant"/>
